Commit message: small changes to camera frame

File: xarm_description/urdf/camera/realsense_d435i.urdf.xacro (robot description, xacro)
@@ -8,10 +8,10 @@
         mesh_filename="camera/realsense/visual/d435_with_cam_stand"
         origin_xyz="0 0 0"
-        origin_rpy="0 0 0"
+        origin_rpy="0 0 ${-M_PI/2}"
         material_name="${prefix}Silver" />
       <xacro:common_link_collision
         mesh_filename="camera/realsense/collision/d435_with_cam_stand"
         origin_xyz="0 0 0"
-        origin_rpy="0 0 0" />
+        origin_rpy="0 0 ${-M_PI/2}" />
     </link>
     <xacro:if value="${add_d435i_links}">
@@ -28,5 +28,9 @@
         <parent link="${prefix}link_eef" />
         <child link="${prefix}camera_link" />
-        <origin xyz="0.06746 -0.0175 0.0237" rpy="${M_PI} ${-M_PI/2} 0" />
+        <!-- nominal mount was xyz="0.015 -0.06 0.03"; shifted by the
+             calibrate_camera_offset delta [0.0022 -0.019 -0.0257] (link_eef
+             frame, 2026-07-24) so the color optical frame lands at the
+             measured [0.0022 -0.079 0.0043] -->
+        <origin xyz="0.0182 -0.0761 0.0061" rpy="${M_PI/2} ${-M_PI/2} 0" />
       </joint>
       <joint name="${prefix}camera_depth_joint" type="fixed">

Commit message: minor offset change for xarm6 robot

File: xarm_description/urdf/camera/realsense_d435i.urdf.xacro (robot description, xacro)
@@ -28,9 +28,6 @@
         <parent link="${prefix}link_eef" />
         <child link="${prefix}camera_link" />
-        <!-- nominal mount was xyz="0.015 -0.06 0.03"; shifted by the
-             calibrate_camera_offset delta [0.0022 -0.019 -0.0257] (link_eef
-             frame, 2026-07-24) so the color optical frame lands at the
-             measured [0.0022 -0.079 0.0043] -->
-        <origin xyz="0.0182 -0.0761 0.0061" rpy="${M_PI/2} ${-M_PI/2} 0" />
+        <!-- For the xarm6Lite <origin xyz="0.0182 -0.0761 0.0061" rpy="${M_PI/2} ${-M_PI/2} 0" /> -->
+        <origin xyz="0.0186 -0.0622 0.0321" rpy="${M_PI/2} ${-M_PI/2} 0" />
       </joint>
       <joint name="${prefix}camera_depth_joint" type="fixed">
