Commit message: minor changes to urdf

File: xarm_description/urdf/lite6/lite6.ros2_control.xacro (robot description, xacro)
@@ -11,5 +11,14 @@
     joint4_lower_limit:=${-2.0*pi}  joint4_upper_limit:=${2.0*pi}
     joint5_lower_limit:=${-2.1642}  joint5_upper_limit:=${2.1642}
-    joint6_lower_limit:=${-2.0*pi}  joint6_upper_limit:=${2.0*pi}">
+    joint6_lower_limit:=${-2.0*pi}  joint6_upper_limit:=${2.0*pi}
+    joint1_home:=0 joint2_home:=${-0.5555} joint3_home:=0
+    joint4_home:=0 joint5_home:=0.5555 joint6_home:=0">
+    <!-- lite6-sim-patches: joint*_home is the pose gz spawns the arm at, via the
+         initial_value params on each position state interface below. It MUST match
+         the 'home' group_state in xarm_moveit_config/srdf/_lite6_macro.srdf.xacro
+         (the all-zero pose lifted 5 cm, so the gripper closing at home clears the
+         floor) — otherwise the arm spawns somewhere RViz's home button will not
+         return it to. Only mock/gz hardware reads initial_value; the real
+         UFRobotSystemHardware plugin reports actual encoder positions. -->
     <ros2_control name="${prefix}${ros2_control_plugin}" type="system">
       <hardware>
@@ -37,5 +46,9 @@
           <param name="max">3.14</param>
         </command_interface>
-        <state_interface name="position"/>
+        <state_interface name="position">
+          <!-- sim start pose; ignored by the real UF plugin (see the
+               joint*_home params above) -->
+          <param name="initial_value">${joint1_home}</param>
+        </state_interface>
         <state_interface name="velocity"/>
         <!-- <state_interface name="effort"/> -->
@@ -50,5 +63,9 @@
           <param name="max">3.14</param>
         </command_interface>
-        <state_interface name="position"/>
+        <state_interface name="position">
+          <!-- sim start pose; ignored by the real UF plugin (see the
+               joint*_home params above) -->
+          <param name="initial_value">${joint2_home}</param>
+        </state_interface>
         <state_interface name="velocity"/>
         <!-- <state_interface name="effort"/> -->
@@ -63,5 +80,9 @@
           <param name="max">3.14</param>
         </command_interface>
-        <state_interface name="position"/>
+        <state_interface name="position">
+          <!-- sim start pose; ignored by the real UF plugin (see the
+               joint*_home params above) -->
+          <param name="initial_value">${joint3_home}</param>
+        </state_interface>
         <state_interface name="velocity"/>
         <!-- <state_interface name="effort"/> -->
@@ -76,5 +97,9 @@
           <param name="max">3.14</param>
         </command_interface>
-        <state_interface name="position"/>
+        <state_interface name="position">
+          <!-- sim start pose; ignored by the real UF plugin (see the
+               joint*_home params above) -->
+          <param name="initial_value">${joint4_home}</param>
+        </state_interface>
         <state_interface name="velocity"/>
         <!-- <state_interface name="effort"/> -->
@@ -89,5 +114,9 @@
           <param name="max">3.14</param>
         </command_interface>
-        <state_interface name="position"/>
+        <state_interface name="position">
+          <!-- sim start pose; ignored by the real UF plugin (see the
+               joint*_home params above) -->
+          <param name="initial_value">${joint5_home}</param>
+        </state_interface>
         <state_interface name="velocity"/>
         <!-- <state_interface name="effort"/> -->
@@ -102,5 +131,9 @@
           <param name="max">3.14</param>
         </command_interface>
-        <state_interface name="position"/>
+        <state_interface name="position">
+          <!-- sim start pose; ignored by the real UF plugin (see the
+               joint*_home params above) -->
+          <param name="initial_value">${joint6_home}</param>
+        </state_interface>
         <state_interface name="velocity"/>
         <!-- <state_interface name="effort"/> -->

File: xarm_description/urdf/xarm6/xarm6.ros2_control.xacro (robot description, xacro)
@@ -11,5 +11,15 @@
     joint4_lower_limit:=${-2.0*pi}  joint4_upper_limit:=${2.0*pi}
     joint5_lower_limit:=${-1.69297}  joint5_upper_limit:=${pi}
-    joint6_lower_limit:=${-2.0*pi}  joint6_upper_limit:=${2.0*pi}">
+    joint6_lower_limit:=${-2.0*pi}  joint6_upper_limit:=${2.0*pi}
+    joint1_home:=0 joint2_home:=${-0.7576} joint3_home:=0.0203
+    joint4_home:=0 joint5_home:=0.7373 joint6_home:=0">
+    <!-- lite6-sim-patches: joint*_home is the pose gz spawns the arm at, via the
+         initial_value params on each position state interface below. It MUST match
+         the 'home' group_state in xarm_moveit_config/srdf/_xarm6_macro.srdf.xacro
+         (the all-zero pose lifted 10 cm — at zeros the stock gripper's link_tcp
+         is 6 cm below the floor, so closing it there drives the fingers into the
+         ground) — otherwise the arm spawns somewhere RViz's home button will not
+         return it to. Only mock/gz hardware reads initial_value; the real
+         UFRobotSystemHardware plugin reports actual encoder positions. -->
     <ros2_control name="${prefix}${ros2_control_plugin}" type="system">
       <hardware>
@@ -44,5 +54,9 @@
           <param name="max">3.14</param>
         </command_interface>
-        <state_interface name="position"/>
+        <state_interface name="position">
+          <!-- sim start pose; ignored by the real UF plugin (see the
+               joint*_home params above) -->
+          <param name="initial_value">${joint1_home}</param>
+        </state_interface>
         <state_interface name="velocity"/>
         <!-- <state_interface name="effort"/> -->
@@ -57,5 +71,9 @@
           <param name="max">3.14</param>
         </command_interface>
-        <state_interface name="position"/>
+        <state_interface name="position">
+          <!-- sim start pose; ignored by the real UF plugin (see the
+               joint*_home params above) -->
+          <param name="initial_value">${joint2_home}</param>
+        </state_interface>
         <state_interface name="velocity"/>
         <!-- <state_interface name="effort"/> -->
@@ -70,5 +88,9 @@
           <param name="max">3.14</param>
         </command_interface>
-        <state_interface name="position"/>
+        <state_interface name="position">
+          <!-- sim start pose; ignored by the real UF plugin (see the
+               joint*_home params above) -->
+          <param name="initial_value">${joint3_home}</param>
+        </state_interface>
         <state_interface name="velocity"/>
         <!-- <state_interface name="effort"/> -->
@@ -83,5 +105,9 @@
           <param name="max">3.14</param>
         </command_interface>
-        <state_interface name="position"/>
+        <state_interface name="position">
+          <!-- sim start pose; ignored by the real UF plugin (see the
+               joint*_home params above) -->
+          <param name="initial_value">${joint4_home}</param>
+        </state_interface>
         <state_interface name="velocity"/>
         <!-- <state_interface name="effort"/> -->
@@ -96,5 +122,9 @@
           <param name="max">3.14</param>
         </command_interface>
-        <state_interface name="position"/>
+        <state_interface name="position">
+          <!-- sim start pose; ignored by the real UF plugin (see the
+               joint*_home params above) -->
+          <param name="initial_value">${joint5_home}</param>
+        </state_interface>
         <state_interface name="velocity"/>
         <!-- <state_interface name="effort"/> -->
@@ -109,5 +139,9 @@
           <param name="max">3.14</param>
         </command_interface>
-        <state_interface name="position"/>
+        <state_interface name="position">
+          <!-- sim start pose; ignored by the real UF plugin (see the
+               joint*_home params above) -->
+          <param name="initial_value">${joint6_home}</param>
+        </state_interface>
         <state_interface name="velocity"/>
         <!-- <state_interface name="effort"/> -->

File: xarm_moveit_config/srdf/_lite6_macro.srdf.xacro (robot description, xacro)
@@ -35,10 +35,20 @@
     </group>
     <!-- GROUP STATES, Purpose, Define a named state for a particular group, in terms of joint values. This is useful to define states like 'folded arms' -->
+    <!-- lite6-sim-patches: home is no longer the all-zero pose. At zeros link6
+         sits at z=0.154 m with the tool pointing straight down, so the custom
+         gripper's jaws reach the floor and closing them there drives them into
+         it (the gripper closes without the arm moving, and the planner cannot
+         back the arm off). This is that pose lifted 5 cm in +z: joint2/joint5
+         pitch by opposite amounts so the tool still points down, and joint3
+         stays at 0 — its lower stop is -0.061087, too close to zero to use for
+         the lateral drift, which is only 1.4 mm anyway. Kept in sync with the
+         initial_value params in xarm_description/urdf/lite6/lite6.ros2_control.xacro
+         so the sim spawns here too. -->
     <group_state name="home" group="${prefix}lite6">
       <joint name="${prefix}joint1" value="0" />
-      <joint name="${prefix}joint2" value="0" />
+      <joint name="${prefix}joint2" value="-0.5555" />
       <joint name="${prefix}joint3" value="0" />
       <joint name="${prefix}joint4" value="0" />
-      <joint name="${prefix}joint5" value="0" />
+      <joint name="${prefix}joint5" value="0.5555" />
       <joint name="${prefix}joint6" value="0" />
     </group_state>

File: xarm_moveit_config/srdf/_xarm6_macro.srdf.xacro (robot description, xacro)
@@ -39,10 +39,23 @@
     </group>
     <!-- GROUP STATES, Purpose, Define a named state for a particular group, in terms of joint values. This is useful to define states like 'folded arms' -->
+    <!-- lite6-sim-patches: home is no longer the all-zero pose. At zeros link6
+         sits at z=0.112 m with the tool pointing straight down, which puts the
+         stock gripper's link_tcp at z=-0.060 — 6 cm INTO the floor. Closing the
+         gripper there drives the fingers through the ground, and nothing can
+         prevent it: the gripper closes without the arm moving, so the planner
+         has no joint to back off.
+         This is that pose lifted 10 cm in +z (link6 0.212, link_tcp +0.040, so
+         ~4 cm of clearance) with x/y and the tool axis unchanged: joint2/joint5
+         pitch by opposite amounts so the tool still points straight down, and
+         joint3 takes up the lateral drift (well inside its 0.19198 upper stop).
+         Kept in sync with the initial_value params in
+         xarm_description/urdf/xarm6/xarm6.ros2_control.xacro so the sim spawns
+         here too. -->
     <group_state name="home" group="${prefix}xarm6">
       <joint name="${prefix}joint1" value="0" />
-      <joint name="${prefix}joint2" value="0" />
-      <joint name="${prefix}joint3" value="0" />
+      <joint name="${prefix}joint2" value="-0.7576" />
+      <joint name="${prefix}joint3" value="0.0203" />
       <joint name="${prefix}joint4" value="0" />
-      <joint name="${prefix}joint5" value="0" />
+      <joint name="${prefix}joint5" value="0.7373" />
       <joint name="${prefix}joint6" value="0" />
     </group_state>
